File: controller.sch (EAGLE design)
At the start: 20 parts, among them IC1 7805TV, Q1 BC639, Q2 BC640, Q3 IRF540, SW1 EC12E_SW

Commit message: Simplify
No encoder (potentiometer now), 2-color led. Working arduino sketch.
Parts:
- removed LED3: (no value), led:LED3MM
- removed R6: 470, resistor:R-EU_0204/7
- removed SW1: EC12E_SW, switch-alps:EC12E_SW
- added R7: 10K, pot:3RP/1610N
Connections:
- removed net N$13: LED3.A, R6.1
- removed net N$14: ARDUINO1.D8, SW1G$1.B
- removed net N$15: ARDUINO1.D9, SW1G$2.1
- removed net N$17: ARDUINO1.D7, SW1G$1.A
- removed net N$18: SW1G$1.C, SW1G$2.2
- net +5V: now also R7.A
- net GND: now also R7.E; no longer LED3.C
- net N$11: now also ARDUINO1.A1, R7.S; no longer ARDUINO1.D6, R6.2
Changed lines of the file:
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@@
 <setting verticaltext="up"/>
 </settings>
-<grid distance="0.1" unitdist="inch" unit="inch" style="lines" multiple="1" display="yes" altdistance="0.01" altunitdist="inch" altunit="inch"/>
+<grid distance="0.1" unitdist="inch" unit="inch" style="lines" multiple="1" display="no" altdistance="0.01" altunitdist="inch" altunit="inch"/>
 <layers>
 <layer number="1" name="Top" color="4" fill="1" visible="no" active="no"/>
@@
 <part name="R4" library="resistor" deviceset="R-EU_" device="0204/7" value="470"/>
 <part name="R5" library="resistor" deviceset="R-EU_" device="0204/7" value="470"/>
-<part name="R6" library="resistor" deviceset="R-EU_" device="0204/7" value="470"/>
 <part name="LED2" library="led" deviceset="LED" device="3MM"/>
-<part name="LED3" library="led" deviceset="LED" device="3MM"/>
 <part name="GND6" library="supply1" deviceset="GND" device=""/>
-<part name="SW1" library="switch-alps" deviceset="EC12E_SW" device=""/>
+<part name="R7" library="pot" deviceset="3RP/1610N" device="" value="10K"/>
+<part name="GND7" library="supply1" deviceset="GND" device=""/>
 </parts>
 <sheets>
@@
 <instance part="R4" gate="G$1" x="-1498.6" y="-93.98" smashed="yes"/>
 <instance part="R5" gate="G$1" x="-1498.6" y="-96.52" smashed="yes"/>
-<instance part="R6" gate="G$1" x="-1498.6" y="-99.06" smashed="yes">
-<attribute name="VALUE" x="-1497.33" y="-102.362" size="1.778" layer="96"/>
-</instance>
 <instance part="LED2" gate="G$1" x="-1508.76" y="-96.52" smashed="yes" rot="R270">
 <attribute name="VALUE" x="-1513.332" y="-102.235" size="1.778" layer="96"/>
 </instance>
-<instance part="LED3" gate="G$1" x="-1513.84" y="-99.06" smashed="yes" rot="R270">
-<attribute name="VALUE" x="-1518.412" y="-104.775" size="1.778" layer="96"/>
-</instance>
-<instance part="GND6" gate="1" x="-1518.92" y="-104.14"/>
-<instance part="SW1" gate="G$1" x="-1506.22" y="-114.3" rot="R270"/>
-<instance part="SW1" gate="G$2" x="-1503.68" y="-129.54"/>
+<instance part="GND6" gate="1" x="-1518.92" y="-101.6"/>
+<instance part="R7" gate="G$1" x="-1442.72" y="-91.44" rot="R180"/>
+<instance part="GND7" gate="1" x="-1442.72" y="-104.14"/>
 </instances>
 <busses>
@@
 <pinref part="R8" gate="G$1" pin="1"/>
 <pinref part="R9" gate="G$1" pin="2"/>
-<wire x1="-1450.34" y1="-53.34" x2="-1440.18" y2="-53.34" width="0.1524" layer="91"/>
-<wire x1="-1440.18" y1="-53.34" x2="-1440.18" y2="-99.06" width="0.1524" layer="91"/>
+<wire x1="-1450.34" y1="-53.34" x2="-1435.1" y2="-53.34" width="0.1524" layer="91"/>
+<wire x1="-1435.1" y1="-53.34" x2="-1435.1" y2="-99.06" width="0.1524" layer="91"/>
 <pinref part="ARDUINO1" gate="G$1" pin="A0"/>
-<wire x1="-1440.18" y1="-99.06" x2="-1452.88" y2="-99.06" width="0.1524" layer="91"/>
+<wire x1="-1435.1" y1="-99.06" x2="-1452.88" y2="-99.06" width="0.1524" layer="91"/>
 <junction x="-1450.34" y="-53.34"/>
 </segment>
@@
 <pinref part="LED2" gate="G$1" pin="C"/>
 <wire x1="-1518.92" y1="-96.52" x2="-1518.92" y2="-99.06" width="0.1524" layer="91"/>
-<wire x1="-1518.92" y1="-99.06" x2="-1518.92" y2="-101.6" width="0.1524" layer="91"/>
 <wire x1="-1518.92" y1="-96.52" x2="-1513.84" y2="-96.52" width="0.1524" layer="91"/>
-<pinref part="LED3" gate="G$1" pin="C"/>
 <pinref part="GND6" gate="1" pin="GND"/>
 <junction x="-1518.92" y="-96.52"/>
-<junction x="-1518.92" y="-99.06"/>
+</segment>
+<segment>
+<pinref part="R7" gate="G$1" pin="E"/>
+<wire x1="-1442.72" y1="-96.52" x2="-1442.72" y2="-101.6" width="0.1524" layer="91"/>
+<pinref part="GND7" gate="1" pin="GND"/>
 </segment>
 </net>
@@
 </segment>
 </net>
-<net name="N$11" class="0">
-<segment>
-<pinref part="ARDUINO1" gate="G$1" pin="D6"/>
-<pinref part="R6" gate="G$1" pin="2"/>
-<wire x1="-1483.36" y1="-99.06" x2="-1493.52" y2="-99.06" width="0.1524" layer="91"/>
-</segment>
-</net>
 <net name="N$12" class="0">
 <segment>
@@
 </segment>
 </net>
-<net name="N$13" class="0">
-<segment>
-<pinref part="LED3" gate="G$1" pin="A"/>
-<pinref part="R6" gate="G$1" pin="1"/>
-<wire x1="-1511.3" y1="-99.06" x2="-1503.68" y2="-99.06" width="0.1524" layer="91"/>
-</segment>
-</net>
 <net name="+5V" class="0">
 <segment>
 <pinref part="ARDUINO1" gate="G$1" pin="VCC"/>
-<wire x1="-1452.88" y1="-78.74" x2="-1422.4" y2="-78.74" width="0.1524" layer="91"/>
+<wire x1="-1452.88" y1="-78.74" x2="-1442.72" y2="-78.74" width="0.1524" layer="91"/>
+<wire x1="-1442.72" y1="-78.74" x2="-1422.4" y2="-78.74" width="0.1524" layer="91"/>
 <wire x1="-1422.4" y1="-78.74" x2="-1422.4" y2="-71.12" width="0.1524" layer="91"/>
 <pinref part="R2" gate="G$1" pin="2"/>
@@
 <wire x1="-1409.7" y1="-71.12" x2="-1402.08" y2="-71.12" width="0.1524" layer="91"/>
 <label x="-1402.08" y="-71.12" size="1.778" layer="95" xref="yes"/>
-<label x="-1508.76" y="-137.16" size="1.778" layer="95" xref="yes"/>
-</segment>
-</net>
-<net name="N$17" class="0">
-<segment>
-<pinref part="ARDUINO1" gate="G$1" pin="D7"/>
-<wire x1="-1488.44" y1="-101.6" x2="-1483.36" y2="-101.6" width="0.1524" layer="91"/>
-<pinref part="SW1" gate="G$1" pin="A"/>
-<wire x1="-1498.6" y1="-111.76" x2="-1488.44" y2="-111.76" width="0.1524" layer="91"/>
-<wire x1="-1488.44" y1="-111.76" x2="-1488.44" y2="-101.6" width="0.1524" layer="91"/>
-</segment>
-</net>
-<net name="N$14" class="0">
-<segment>
-<pinref part="SW1" gate="G$1" pin="B"/>
-<wire x1="-1498.6" y1="-116.84" x2="-1485.9" y2="-116.84" width="0.1524" layer="91"/>
-<wire x1="-1485.9" y1="-116.84" x2="-1485.9" y2="-104.14" width="0.1524" layer="91"/>
-<pinref part="ARDUINO1" gate="G$1" pin="D8"/>
-<wire x1="-1485.9" y1="-104.14" x2="-1483.36" y2="-104.14" width="0.1524" layer="91"/>
-</segment>
-</net>
-<net name="N$15" class="0">
-<segment>
-<pinref part="ARDUINO1" gate="G$1" pin="D9"/>
-<wire x1="-1483.36" y1="-106.68" x2="-1483.36" y2="-119.38" width="0.1524" layer="91"/>
-<wire x1="-1483.36" y1="-119.38" x2="-1496.06" y2="-119.38" width="0.1524" layer="91"/>
-<wire x1="-1496.06" y1="-119.38" x2="-1496.06" y2="-129.54" width="0.1524" layer="91"/>
-<pinref part="SW1" gate="G$2" pin="1"/>
-<wire x1="-1496.06" y1="-129.54" x2="-1498.6" y2="-129.54" width="0.1524" layer="91"/>
-</segment>
-</net>
-<net name="N$18" class="0">
-<segment>
-<pinref part="SW1" gate="G$1" pin="C"/>
-<wire x1="-1508.76" y1="-114.3" x2="-1511.3" y2="-114.3" width="0.1524" layer="91"/>
-<wire x1="-1511.3" y1="-114.3" x2="-1511.3" y2="-129.54" width="0.1524" layer="91"/>
-<pinref part="SW1" gate="G$2" pin="2"/>
-<wire x1="-1511.3" y1="-129.54" x2="-1511.3" y2="-137.16" width="0.1524" layer="91"/>
-<wire x1="-1511.3" y1="-129.54" x2="-1508.76" y2="-129.54" width="0.1524" layer="91"/>
-<junction x="-1511.3" y="-129.54"/>
-<wire x1="-1511.3" y1="-137.16" x2="-1508.76" y2="-137.16" width="0.1524" layer="91"/>
-</segment>
-</net>
+<pinref part="R7" gate="G$1" pin="A"/>
+<wire x1="-1442.72" y1="-86.36" x2="-1442.72" y2="-78.74" width="0.1524" layer="91"/>
+<junction x="-1442.72" y="-78.74"/>
+</segment>
+</net>
+<net name="N$11" class="0">
+<segment>
+<pinref part="ARDUINO1" gate="G$1" pin="A1"/>
+<pinref part="R7" gate="G$1" pin="S"/>
+<wire x1="-1452.88" y1="-96.52" x2="-1447.8" y2="-96.52" width="0.1524" layer="91"/>
+<wire x1="-1447.8" y1="-96.52" x2="-1447.8" y2="-91.44" width="0.1524" layer="91"/>
+</segment>
+</net>
